File: Hardware/Wisol-Breakout.brd (EAGLE design)
At the start: 21.6 x 25.4 mm, 15 parts

Commit message: Added annotations for Wisol WSSFM10R H/W Design Guide
Connections:
- removed net GPIO1: WSSFM10R.24
- removed net GPIO2: WSSFM10R.25
Changed lines of the file:
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@@
 <wire x1="48.82899375" y1="44.5175" x2="48.846146875" y2="44.534653125" width="0.254" layer="1"/>
-</signal>
-<signal name="GPIO2">
-<contactref element="WSSFM10R" pad="25"/>
-</signal>
-<signal name="GPIO1">
-<contactref element="WSSFM10R" pad="24"/>
 </signal>
 <signal name="N$4">
